File: KiCad/Senior Project.kicad_sch (KiCad schematic)
At the start: 29 parts, among them J1 USB_C_Receptacle_USB2.0_16P, J2 Screw_Terminal_01x02, J3 Screw_Terminal_01x06, SW1 SW_Push, SW2 SW_Push, U1 ESP32-S3FH4R2, X1 FC-135 32.7680KA-A5, Y2 Crystal_GND23

Commit message: Added diode footprint
Parts:
- D1: footprint (none) -> Diode_PCB:DO-41_STM
Changed lines of the file:
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@@
 			)
 		)
-		(property "Footprint" ""
+		(property "Footprint" "Diode_PCB:DO-41_STM"
 			(at 69.85 44.45 0)
 			(effects
@@
 			)
 		)
-		(property "Datasheet" "~"
+		(property "Datasheet" "~https://www.st.com/content/ccc/resource/technical/document/datasheet/26/db/14/60/52/47/47/5b/CD00001625.pdf/files/CD00001625.pdf/jcr:content/translations/en.CD00001625.pdf"
 			(at 69.85 44.45 0)
 			(effects
